Commit message: lidar avance intermedio

File: robot/description/lidar.xacro (robot description, xacro)
@@ -2,7 +2,7 @@
 <robot xmlns:xacro="http://www.ros.org/wiki/xacro" >
     <joint name="laser_joint" type="fixed">
-        <parent link="chassis"/>
+        <parent link="chassis2"/>
         <child link="laser_frame"/>
-        <origin xyz="0.1 0 0.175" rpy="0 0 0"/>
+        <origin xyz="0.17 0 0.155" rpy="0 0 0"/>
     </joint>
     <link name="laser_frame">

File: robot/description/robot_core.xacro (robot description, xacro)
@@ -16,4 +16,12 @@
     <!-- BASE LINK -->
     <link name="base_link">
+    </link>
+    <!-- BASE_FOOTPRINT LINK -->
+    <joint name="base_footprint_joint" type="fixed">
+        <parent link="base_link"/>
+        <child link="base_footprint"/>
+        <origin xyz="0 0 0" rpy="0 0 0"/>
+    </joint>
+    <link name="base_footprint">
     </link>
     <!-- CHASSIS LINK -->

Commit message: correccion timestamp

File: robot/description/lidar.xacro (robot description, xacro)
@@ -1,4 +1,7 @@
 <?xml version="1.0"?>
 <robot xmlns:xacro="http://www.ros.org/wiki/xacro" >
+    <material name="red">
+        <color rgba="1 0 0 1"/>
+    </material>
     <joint name="laser_joint" type="fixed">
         <parent link="chassis2"/>
