Commit message: fix saltos mapeo; cartogrp no anda

File: robot/description/robot_core.xacro (robot description, xacro)
@@ -76,5 +76,5 @@
         <parent link="base_link"/>
         <child link="left_wheel"/>
-        <origin xyz="0 0.207 0" rpy="-${pi/2} 0 0" />
+        <origin xyz="0 0.204 0" rpy="-${pi/2} 0 0" />
         <axis xyz="0 0 1"/>
     </joint>
@@ -99,5 +99,5 @@
         <parent link="base_link"/>
         <child link="right_wheel"/>
-        <origin xyz="0 -0.207 0" rpy="${pi/2} 0 0" />
+        <origin xyz="0 -0.204 0" rpy="${pi/2} 0 0" />
         <axis xyz="0 0 -1"/>
     </joint>
