Commit message: full simulations with the new gzebo Fortress

File: robot/description/imu.xacro (robot description, xacro)
@@ -7,6 +7,7 @@
         <parent link="chassis2"/>
         <child link="imu_frame"/>
-        <origin xyz="0.14 0.1 0.12" rpy="0 0 0"/>
+        <origin xyz="0.14 0.1 0.155" rpy="0 0 0"/>
     </joint>
+    <!-- Sin <collision> (link de sensor). -->
     <link name="imu_frame">
         <visual>
@@ -17,12 +18,16 @@
             <!-- <material name="red"/> -->
         </visual>
-        <collision>
-            <geometry>
-                <box size="0.02 0.01 0.01"/>
-            </geometry>
-        </collision>
         <xacro:inertial_box mass="0.1" x="0.02" y="0.01" z="0.01">
             <origin xyz="0.14 0.1 0.155" rpy="0 0 0"/>
         </xacro:inertial_box>
     </link>
+    <!-- Gazebo Fortress: el topics gz "imu/data_raw"; ros_gz_bridge como /imu/data_raw -->
+    <gazebo reference="imu_frame">
+        <sensor name="imu_sensor" type="imu">
+            <topic>imu/data_raw</topic>
+            <ignition_frame_id>imu_frame</ignition_frame_id>
+            <update_rate>100</update_rate>
+            <always_on>1</always_on>
+        </sensor>
+    </gazebo>
 </robot>

File: robot/description/lidar.xacro (robot description, xacro)
@@ -7,5 +7,5 @@
         <parent link="chassis2"/>
         <child link="laser_frame"/>
-        <origin xyz="0.17 0 0.155" rpy="0 0 0"/>
+        <origin xyz="0.17 0 0.19" rpy="0 0 0"/>
     </joint>
     <link name="laser_frame">
@@ -16,40 +16,32 @@
             <material name="red"/>
         </visual>
-        <collision>
-            <geometry>
-                <cylinder radius="0.05" length="0.07"/>
-            </geometry>
-        </collision>
         <xacro:inertial_cylinder mass="0.1" length="0.07" radius="0.05">
             <origin xyz="0 0 0" rpy="0 0 0"/>
         </xacro:inertial_cylinder>
     </link>
-    <!-- <gazebo reference="laser_frame">
-        <material>Gazebo/Red</material>
-        <sensor name="laser" type="ray">
-            <pose> 0 0 0 0 0 0 </pose>
+    <!-- Gazebo Fortress:
+         topic gz "scan"; ros_gz_bridge lo trae a ROS como /scan. -->
+    <gazebo reference="laser_frame">
+        <sensor name="laser" type="gpu_lidar">
+            <pose>0 0 0 0 0 0</pose>
+            <topic>scan</topic>
+            <ignition_frame_id>laser_frame</ignition_frame_id>
+            <update_rate>7</update_rate>
+            <always_on>1</always_on>
             <visualize>true</visualize>
-            <update_rate>10</update_rate>
-            <ray>
+            <lidar>
                 <scan>
                     <horizontal>
                         <samples>360</samples>
-                        <min_angle>-3.14</min_angle>
-                        <max_angle>3.14</max_angle>
+                        <min_angle>-3.14159</min_angle>
+                        <max_angle>3.14159</max_angle>
                     </horizontal>
                 </scan>
                 <range>
-                    <min>0.3</min>
-                    <max>12</max>
+                    <min>0.16</min>
+                    <max>6.0</max>
                 </range>
-            </ray>
-            <plugin name="laser_controller" filename="libgazebo_ros_ray_sensor.so">
-                <ros>
-                    <argument>~/out:=scan</argument>
-                </ros>
-                <output_type>sensor_msgs/LaserScan</output_type>
-                <frame_name>laser_frame</frame_name>
-            </plugin>
+            </lidar>
         </sensor>
-    </gazebo> -->
+    </gazebo>
 </robot>

File: robot/description/robot.urdf.xacro (robot description, xacro)
@@ -1,6 +1,11 @@
 <?xml version="1.0"?>
 <robot xmlns:xacro="http://www.ros.org/wiki/xacro"  name="robot">
+    <xacro:arg name="sim_mode" default="false"/>
     <xacro:include filename="robot_core.xacro" />
     <xacro:include filename="ros2_control.xacro" />
+    <!-- Plugin gazebo_ros2_control: solo en simulación -->
+    <xacro:if value="$(arg sim_mode)">
+        <xacro:include filename="gazebo_control.xacro" />
+    </xacro:if>
     <xacro:include filename="lidar.xacro" />
     <xacro:include filename="imu.xacro" />

File: robot/description/robot_core.xacro (robot description, xacro)
@@ -56,5 +56,5 @@
     <link name="chassis2">
         <visual>
-            <origin xyz="0.11 0 0.06"/>
+            <origin xyz="0.11 0 0.095"/>
             <geometry>
                 <box size="0.22 0.22 0.12"/>
@@ -63,5 +63,5 @@
         </visual>
         <collision>
-            <origin xyz="0.11 0 0.06"/>
+            <origin xyz="0.11 0 0.095"/>
             <geometry>
                 <box size="0.22 0.22 0.12"/>
@@ -69,5 +69,5 @@
         </collision>
         <xacro:inertial_box mass="0.4" x="0.22" y="0.22" z="0.12">
-            <origin xyz="0.11 0 0.06" rpy="0 0 0"/>
+            <origin xyz="0.11 0 0.095" rpy="0 0 0"/>
         </xacro:inertial_box>
     </link>
@@ -140,3 +140,7 @@
         </xacro:inertial_sphere>
     </link>
+    <gazebo reference="caster_wheel">
+        <mu1>0.001</mu1>
+        <mu2>0.001</mu2>
+    </gazebo>
 </robot>

File: robot/description/ros2_control.xacro (robot description, xacro)
@@ -1,22 +1,30 @@
 <?xml version="1.0"?>
 <robot xmlns:xacro="http://www.ros.org/wiki/xacro">
+    <!-- sim_mode=true intercambia el plugin de hardware real por el de Gazebo.
+         Se reutilizan los mismos <joint> y la misma config de controllers. -->
+    <xacro:arg name="sim_mode" default="false"/>
     <ros2_control name="RealRobot" type="system">
         <hardware>
-            <plugin>diffdrive_arduino/DiffDriveArduinoHardware</plugin>
-            <param name="left_wheel_name">left_wheel_joint</param>
-            <param name="right_wheel_name">right_wheel_joint</param>
-            <param name="loop_rate">100</param>
-            <param name="device">/dev/serial/by-id/usb-Espressif_USB_JTAG_serial_debug_unit_10:20:BA:4D:92:80-if00</param>
-            <param name="baud_rate">57600</param>
-            <param name="timeout_ms">100</param>
-            <!-- <param name="enc_counts_per_rev_left">33572</param> -->
-            <!-- <param name="enc_counts_per_rev_right">32730</param> -->
-            <param name="enc_counts_per_rev_left">33667</param>
-            <param name="enc_counts_per_rev_right">41800</param>
-            <!-- Sensor de batería (opcional, valores por defecto en el código) -->
-            <param name="battery_voltage_min">10.75</param>
-            <param name="battery_voltage_max">12.6</param>
-            <param name="battery_runtime_full_min">120.0</param>
-            <param name="battery_publish_period">60.0</param>
+            <xacro:unless value="$(arg sim_mode)">
+                <plugin>diffdrive_arduino/DiffDriveArduinoHardware</plugin>
+                <param name="left_wheel_name">left_wheel_joint</param>
+                <param name="right_wheel_name">right_wheel_joint</param>
+                <param name="loop_rate">100</param>
+                <param name="device">/dev/serial/by-id/usb-Espressif_USB_JTAG_serial_debug_unit_10:20:BA:4D:92:80-if00</param>
+                <param name="baud_rate">57600</param>
+                <param name="timeout_ms">100</param>
+                <!-- <param name="enc_counts_per_rev_left">33572</param> -->
+                <!-- <param name="enc_counts_per_rev_right">32730</param> -->
+                <param name="enc_counts_per_rev_left">33667</param>
+                <param name="enc_counts_per_rev_right">41800</param>
+                <!-- Sensor de batería (opcional, valores por defecto en el código) -->
+                <param name="battery_voltage_min">10.75</param>
+                <param name="battery_voltage_max">12.6</param>
+                <param name="battery_runtime_full_min">120.0</param>
+                <param name="battery_publish_period">60.0</param>
+            </xacro:unless>
+            <xacro:if value="$(arg sim_mode)">
+                <plugin>ign_ros2_control/IgnitionSystem</plugin>
+            </xacro:if>
         </hardware>
         <joint name="left_wheel_joint">

Commit message: fix comments and update battery sensor

File: robot/description/imu.xacro (robot description, xacro)
@@ -1,7 +1,4 @@
 <?xml version="1.0"?>
 <robot xmlns:xacro="http://www.ros.org/wiki/xacro" >
-    <!-- <material name="red">
-        <color rgba="1 0 0 1"/>
-    </material> -->
     <joint name="imu_joint" type="fixed">
         <parent link="chassis2"/>
@@ -9,5 +6,4 @@
         <origin xyz="0.14 0.1 0.155" rpy="0 0 0"/>
     </joint>
-    <!-- Sin <collision> (link de sensor). -->
     <link name="imu_frame">
         <visual>
@@ -16,5 +12,4 @@
             </geometry>
             <color rgba="1 0 0 1"/>
-            <!-- <material name="red"/> -->
         </visual>
         <xacro:inertial_box mass="0.1" x="0.02" y="0.01" z="0.01">
@@ -22,5 +17,4 @@
         </xacro:inertial_box>
     </link>
-    <!-- Gazebo Fortress: el topics gz "imu/data_raw"; ros_gz_bridge como /imu/data_raw -->
     <gazebo reference="imu_frame">
         <sensor name="imu_sensor" type="imu">

File: robot/description/lidar.xacro (robot description, xacro)
@@ -20,6 +20,4 @@
         </xacro:inertial_cylinder>
     </link>
-    <!-- Gazebo Fortress:
-         topic gz "scan"; ros_gz_bridge lo trae a ROS como /scan. -->
     <gazebo reference="laser_frame">
         <sensor name="laser" type="gpu_lidar">

File: robot/description/robot.urdf.xacro (robot description, xacro)
@@ -4,5 +4,5 @@
     <xacro:include filename="robot_core.xacro" />
     <xacro:include filename="ros2_control.xacro" />
-    <!-- Plugin gazebo_ros2_control: solo en simulación -->
+    <!-- Plugin gazebo_ros2_control solo en simulación -->
     <xacro:if value="$(arg sim_mode)">
         <xacro:include filename="gazebo_control.xacro" />

File: robot/description/ros2_control.xacro (robot description, xacro)
@@ -1,5 +1,5 @@
 <?xml version="1.0"?>
 <robot xmlns:xacro="http://www.ros.org/wiki/xacro">
-    <!-- sim_mode=true intercambia el plugin de hardware real por el de Gazebo.
+    <!-- sim_mode=true intercambia el plugin de hardware real por el de Gazebo
          Se reutilizan los mismos <joint> y la misma config de controllers. -->
     <xacro:arg name="sim_mode" default="false"/>
@@ -18,7 +18,7 @@
                 <param name="enc_counts_per_rev_left">33667</param>
                 <param name="enc_counts_per_rev_right">41800</param>
-                <!-- Sensor de batería (opcional, valores por defecto en el código) -->
-                <param name="battery_voltage_min">10.75</param>
-                <param name="battery_voltage_max">12.6</param>
+                <!-- Sensor de bateria -->
+                <param name="battery_voltage_min">12.0</param>
+                <param name="battery_voltage_max">16.8</param>
                 <param name="battery_runtime_full_min">120.0</param>
                 <param name="battery_publish_period">60.0</param>

Commit message: fix real dimensions

File: robot/description/imu.xacro (robot description, xacro)
@@ -4,5 +4,5 @@
         <parent link="chassis2"/>
         <child link="imu_frame"/>
-        <origin xyz="0.14 0.1 0.155" rpy="0 0 0"/>
+        <origin xyz="0.177 0.067 0.004" rpy="0 0 0"/>
     </joint>
     <link name="imu_frame">
@@ -11,9 +11,8 @@
                 <box size="0.02 0.01 0.01"/>
             </geometry>
-            <color rgba="1 0 0 1"/>
+            <material name="red">
+                <color rgba="1 0 0 1"/>
+            </material>
         </visual>
-        <xacro:inertial_box mass="0.1" x="0.02" y="0.01" z="0.01">
-            <origin xyz="0.14 0.1 0.155" rpy="0 0 0"/>
-        </xacro:inertial_box>
     </link>
     <gazebo reference="imu_frame">

File: robot/description/lidar.xacro (robot description, xacro)
@@ -1,20 +1,21 @@
 <?xml version="1.0"?>
 <robot xmlns:xacro="http://www.ros.org/wiki/xacro" >
-    <material name="red">
-        <color rgba="1 0 0 1"/>
-    </material>
     <joint name="laser_joint" type="fixed">
         <parent link="chassis2"/>
         <child link="laser_frame"/>
-        <origin xyz="0.17 0 0.19" rpy="0 0 0"/>
+        <!-- <origin xyz="0.17 0 0.19" rpy="0 0 0"/> -->
+        <origin xyz="0.114 0 0.15" rpy="0 0 0"/>
     </joint>
     <link name="laser_frame">
         <visual>
             <geometry>
-                <cylinder radius="0.05" length="0.07"/>
+                <!-- <cylinder radius="0.05" length="0.07"/> -->
+                <cylinder radius="0.05" length="0.024"/>
             </geometry>
-            <material name="red"/>
+            <material name="red">
+                <color rgba="1 0 0 1"/>
+            </material>
         </visual>
-        <xacro:inertial_cylinder mass="0.1" length="0.07" radius="0.05">
+        <xacro:inertial_cylinder mass="0.1" length="0.024" radius="0.05">
             <origin xyz="0 0 0" rpy="0 0 0"/>
         </xacro:inertial_cylinder>

File: robot/description/robot_core.xacro (robot description, xacro)
@@ -2,16 +2,5 @@
 <robot xmlns:xacro="http://www.ros.org/wiki/xacro" >
     <xacro:include filename="inertial_macros.xacro"/>
-    <material name="white">
-        <color rgba="0.5 0.5 0.5 1" />
-    </material>
-    <material name="orange">
-        <color rgba="1 0.3 0.1 1"/>
-    </material>
-    <material name="blue">
-        <color rgba="0.2 0.2 1 1"/>
-    </material>
-    <material name="black">
-        <color rgba="0 0 0 1"/>
-    </material>
+    <!-- Gazebo Fortress mapea (URDF-SDF) colores a diffuse/ambient -->
     <!-- BASE LINK -->
     <link name="base_link">
@@ -29,21 +18,23 @@
         <parent link="base_link"/>
         <child link="chassis1"/>
-        <origin xyz="-0.05 0 -0.045"/>
+        <origin xyz="-0.047 0 -0.046"/>
     </joint>
     <link name="chassis1">
         <visual>
-            <origin xyz="0.05 0 0.1"/>
+            <origin xyz="0.047 0 0.1"/>
             <geometry>
-                <box size="0.1 0.38 0.2"/>
+                <box size="0.094 0.354 0.2"/>
             </geometry>
-            <material name="white"/>
+            <material name="gray">
+                <color rgba="0.35 0.35 0.35 1"/>
+            </material>
         </visual>
         <collision>
-            <origin xyz="0.05 0 0.1"/>
+            <origin xyz="0.047 0 0.1"/>
             <geometry>
-                <box size="0.1 0.38 0.2"/>
+                <box size="0.094 0.354 0.2"/>
             </geometry>
         </collision>
-        <xacro:inertial_box mass="0.6" x="0.1" y="0.38" z="0.2">
+        <xacro:inertial_box mass="0.6" x="0.094" y="0.354" z="0.2">
             <origin xyz="0.05 0 0.1" rpy="0 0 0"/>
         </xacro:inertial_box>
@@ -52,16 +43,20 @@
         <parent link="base_link"/>
         <child link="chassis2"/>
-        <origin xyz="0.05 0 0"/>
+        <origin xyz="0.065 0 0.024"/>
     </joint>
     <link name="chassis2">
         <visual>
-            <origin xyz="0.11 0 0.095"/>
+            <!-- <origin xyz="0.11 0 0.095"/> -->
+            <origin xyz="0.098 0 0.055"/>
             <geometry>
-                <box size="0.22 0.22 0.12"/>
+                <box size="0.196 0.156 0.11"/>
             </geometry>
-            <material name="white"/>
+            <material name="gray">
+                <color rgba="0.35 0.35 0.35 1"/>
+            </material>
         </visual>
         <collision>
-            <origin xyz="0.11 0 0.095"/>
+            <!-- <origin xyz="0.11 0 0.095"/> -->
+            <origin xyz="0.098 0 0.055"/>
             <geometry>
                 <box size="0.22 0.22 0.12"/>
@@ -69,5 +64,5 @@
         </collision>
         <xacro:inertial_box mass="0.4" x="0.22" y="0.22" z="0.12">
-            <origin xyz="0.11 0 0.095" rpy="0 0 0"/>
+            <origin xyz="0.098 0 0.055" rpy="0 0 0"/>
         </xacro:inertial_box>
     </link>
@@ -82,14 +77,16 @@
         <visual>
             <geometry>
-                <cylinder radius="0.055" length="0.025"/>
+                <cylinder radius="0.056" length="0.027"/>
             </geometry>
-            <material name="blue"/>
+            <material name="blue">
+                <color rgba="0.2 0.2 1 1"/>
+            </material>
         </visual>
         <collision>
             <geometry>
-                <cylinder radius="0.055" length="0.025"/>
+                <cylinder radius="0.056" length="0.027"/>
             </geometry>
         </collision>
-        <xacro:inertial_cylinder mass="0.05" length="0.025" radius="0.055">
+        <xacro:inertial_cylinder mass="0.05" length="0.027" radius="0.056">
             <origin xyz="0 0 0" rpy="0 0 0"/>
         </xacro:inertial_cylinder>
@@ -105,14 +102,16 @@
         <visual>
             <geometry>
-                <cylinder radius="0.055" length="0.025"/>
+                <cylinder radius="0.056" length="0.027"/>
             </geometry>
-            <material name="blue"/>
+            <material name="blue">
+                <color rgba="0.2 0.2 1 1"/>
+            </material>
         </visual>
         <collision>
             <geometry>
-                <cylinder radius="0.055" length="0.025"/>
+                <cylinder radius="0.056" length="0.027"/>
             </geometry>
         </collision>
-        <xacro:inertial_cylinder mass="0.05" length="0.025" radius="0.055">
+        <xacro:inertial_cylinder mass="0.05" length="0.027" radius="0.056">
             <origin xyz="0 0 0" rpy="0 0 0"/>
         </xacro:inertial_cylinder>
@@ -122,19 +121,21 @@
         <parent link="chassis2"/>
         <child link="caster_wheel"/>
-        <origin xyz="0.165 0 0"/>
+        <origin xyz="0.156 0 -0.024"/>
     </joint>
     <link name="caster_wheel">
         <visual>
             <geometry>
-                <sphere radius="0.055"/>
+                <sphere radius="0.056"/>
             </geometry>
-            <material name="white"/>
+            <material name="white">
+                <color rgba="0.5 0.5 0.5 1"/>
+            </material>
         </visual>
         <collision>
             <geometry>
-                <sphere radius="0.055"/>
+                <sphere radius="0.056"/>
             </geometry>
         </collision>
-        <xacro:inertial_sphere mass="0.02" radius="0.055">
+        <xacro:inertial_sphere mass="0.02" radius="0.056">
             <origin xyz="0 0 0" rpy="0 0 0"/>
         </xacro:inertial_sphere>
